Commit message: More progress towards getting the hardware interface rewritten

File: description/urdf/amy_marks.urdf.xacro (robot description, xacro)
@@ -4,7 +4,4 @@
   <xacro:include filename="$(find happy)/ros2_control/happy.ros2_control.xacro" />
   <!--All units in m-kg-s-radians unit system -->
-  <xacro:property name="M_PI" value="3.1415926535897931" />
-  <xacro:property name="PI_2" value="1.5707963267949" />
-  <xacro:property name="DEG_TO_RAD" value="0.017453293" />
   <xacro:macro name="box_inertia" params="m x y z">
   <inertia  ixx="${m*(y*y+z*z)/12}" ixy = "0" ixz = "0"
@@ -18,4 +15,21 @@
   </xacro:sick_tim551>
   <link name="dummy">
+  </link>
+  <joint name="chassis_joint" type="fixed">
+    <parent link="base_link" />
+    <child link="chassis" />
+    <origin xyz="-0.1 0 0"/>
+  </joint>
+  <link name="chassis">
+    <collision>
+      <origin xyz="0.1 0 0.05" />
+      <geometry>
+        <box size="-0.69 -0.55 0.24"/>
+      </geometry>
+      <material name="">
+        <color
+          rgba="1 1 1 1" />
+      </material>
+    </collision>
   </link>
   <joint name="dummy_joint" type="fixed">
@@ -41,5 +55,5 @@
       <origin
         xyz="0 0 0"
-        rpy="1.5707963267949 0 1.5707963267949" />
+        rpy="-${pi/2} 0 -${pi/2}" />
       <geometry>
         <mesh
@@ -55,5 +69,5 @@
       <origin
         xyz="0 0 0"
-        rpy="1.5707963267949 0 1.5707963267949" />
+        rpy="-${pi/2} 0 -${pi/2}" />
       <geometry>
         <mesh
@@ -81,5 +95,5 @@
       <origin
         xyz="0 0 0"
-        rpy="1.5707963267949 0 1.5707963267949" />
+        rpy="-${pi/2} 0 -${pi/2}" />
       <geometry>
         <mesh
@@ -95,5 +109,5 @@
       <origin
         xyz="0 0 0"
-        rpy="1.5707963267949 0 1.5707963267949" />
+        rpy="-${pi/2} 0 -${pi/2}" />
       <geometry>
         <mesh
@@ -104,5 +118,5 @@
   <joint
     name="lwheel_to_base"
-    type="fixed">
+    type="continuous">
     <origin
       xyz="0 0.241 -0.040"
@@ -113,5 +127,5 @@
       link="lwheel" />
     <axis
-      xyz="0 0 0" />
+      xyz="0 1 0" />
   </joint>
   <link
@@ -134,5 +148,5 @@
       <origin
         xyz="0 0 0"
-        rpy="1.5707963267949 0 1.5707963267949" />
+        rpy="-${pi/2} 0 -${pi/2}" />
       <geometry>
         <mesh
@@ -148,5 +162,5 @@
       <origin
         xyz="0 0 0"
-        rpy="1.5707963267949 0 1.5707963267949" />
+        rpy="-${pi/2} 0 -${pi/2}" />
       <geometry>
         <mesh
@@ -157,5 +171,5 @@
   <joint
     name="rwheel_to_base"
-    type="fixed">
+    type="continuous">
     <origin
       xyz="0 -0.241 -0.040"
@@ -166,5 +180,5 @@
       link="rwheel" />
     <axis
-      xyz="0 0 0" />
+      xyz="0 1 0" />
   </joint>
   <link name="sonar1">
@@ -184,5 +198,5 @@
     <origin
       xyz="-0.31098 -0.26401 0.0243"
-      rpy="0 0 3.92699075" />
+      rpy="0 0 ${pi * 1.25}" />
     <parent
       link="base_link" />
@@ -208,5 +222,5 @@
     <origin
       xyz="-0.345 0 0.0243"
-      rpy="0 0 3.1415926" />
+      rpy="0 0 ${pi}" />
     <parent
       link="base_link" />
@@ -232,5 +246,5 @@
     <origin
       xyz="-0.31098 0.26401 0.0243"
-      rpy="0 0 2.35619445" />
+      rpy="0 0 ${0.75 * pi}" />
     <parent
       link="base_link" />
@@ -256,5 +270,5 @@
     <origin
       xyz="0.31098 0.26401 0.0243"
-      rpy="0 0 0.78539815" />
+      rpy="0 0 ${0.25 * pi}" />
     <parent
       link="base_link" />
@@ -304,5 +318,5 @@
     <origin
       xyz="0.345 -0.26401 0.0243"
-      rpy="0 0 5.42247" />
+      rpy="0 0 ${1.75 * pi}" />
     <parent
       link="base_link" />
@@ -312,51 +326,3 @@
       xyz="0 0 0" />
   </joint>
-  <link name="camera_link">
-    <visual>
-      <geometry>
-        <box size="0.01 0.02 0.01"/>
-      </geometry>
-      <origin rpy="0 0 0" xyz="0.0 0 0.0"/>
-      <material name="blue">
-        <color rgba="0 0 .8 1"/>
-      </material>
-    </visual>
-  </link>
-  <joint
-    name="AXONcamera_to_base"
-    type="fixed">
-    <origin
-      xyz="0.345 0 0.1943"
-      rpy="0 0 0" />
-    <parent
-      link="base_link" />
-    <child
-      link="camera_link" />
-    <axis
-      xyz="0 0 0" />
-  </joint>
-    <link name="sonarScan">
-    <visual>
-      <geometry>
-        <box size="0.01 0.02 0.01"/>
-      </geometry>
-      <origin rpy="0 0 0" xyz="0.0 0 0.0"/>
-      <material name="blue">
-        <color rgba="0 0 .8 1"/>
-      </material>
-    </visual>
-  </link>
-  <joint
-     name="sonarScan_to_base"
-     type="fixed">
-    <origin
-      xyz="0 0 0.29928"
-      rpy="0 0 0" />
-    <parent
-      link="base_link" />
-    <child
-      link="sonarScan" />
-    <axis
-      xyz="0 0 0" />
-  </joint>
 </robot>
